Commit message: Funciona hardware interface ( simple )

File: bots_description/ackerman/urdf/ackerman.urdf.xacro (robot description, xacro)
@@ -10,6 +10,8 @@
   <xacro:property name="PI" value="3.14159265359"/>
   <!-- Chasis -->
-  <link name="base_link">
-    <visual>
+  <link name="base_link"/>
+<!-- chasis link -->
+  <link name="chasis_link">
+      <visual>
       <geometry>
         <box size="${wheelbase} ${wheel_separation} 0.1"/>
@@ -28,4 +30,9 @@
     </inertial>
   </link>
+  <joint name="chasis_joint" type="fixed">
+    <parent link="base_link"/>
+    <child link="chasis_link"/>
+    <origin xyz="0 0 0" rpy="0 0 0"/>
+  </joint>
   <!-- Ruedas Traseras -->
   <link name="left_rear_wheel">
